File: M5stamp_round_lcd.brd (EAGLE design)
At the start: 36 x 38.1 mm, 11 parts, among them Q1 200mA/50V, U1 M5STAMP_C3U_MATE, U2 ROUND_IPS_LCD

Commit message: Add files via upload
Parts:
- removed J1: (no value), SparkFun-Connectors:1X06
- removed U$1: (no value), sunalogo:HYOUTAN
- added F1: F0603E0R25FSTR, suna_lib:C0603
- added TP1, TP2, TP3, TP4, TP5, TP6, TP7: TPTP18R, testpad:TP18R
- R6: value N.C -> 100
Connections:
- new net N$3: F1.2, U2.3, U2.4
- net +3V3: now also F1.1, TP7.TP; no longer U2.4
- net 5V: now also TP6.TP; no longer J1.6, U2.3
- net G20: now also TP2.TP; no longer J1.2
- net G21: now also TP3.TP; no longer J1.3
- net GND: now also TP1.TP; no longer J1.1
- net SCL: now also TP5.TP; no longer J1.5
- net SDA: now also TP4.TP; no longer J1.4
Routing:
- net N$3: track 0.00 -> 24.4 mm, vias 0 -> 1
- net 5V: track 67.9 -> 58.1 mm
- net LCD_DI: track 31.5 -> 24.0 mm, vias 1 -> 3
- net LCD_CS: track 16.4 -> 23.0 mm, vias 3 -> 1
- net SCL: track 23.6 -> 28.3 mm, vias 0 -> 2
- net SDA: track 34.6 -> 38.0 mm
- net G21: track 6.65 -> 8.67 mm
- net LEDK: track 28.0 -> 26.6 mm
- net G20: track 6.59 -> 7.78 mm
- net LCD_RESET: track 17.0 -> 18.2 mm
- net LCD_DC: track 12.9 -> 14.1 mm
- net LED_EN: track 3.59 -> 4.39 mm
- net +3V3: track 33.6 -> 33.8 mm, vias 1 -> 2
Other:
- board text added: "3.3V"
- board text added: "Ver1.2"
- board text removed: "Ver1.0"
