File: M5stamp_round_lcd.sch (EAGLE design)
At the start: 10 parts, among them Q1 200mA/50V, U1 M5STAMP_C3U_MATE, U2 ROUND_IPS_LCD

Commit message: Add files via upload
Parts:
- removed J1: (no value), SparkFun-Connectors:CONN_06SILK_FEMALE_PTH
- added F1: F0603E0R25FSTR, suna_lib:FUSE0603
- added TP1, TP2, TP3, TP4, TP5, TP6, TP7: TPTP18R, testpad:TPTP18R
- R6: value N.C -> 100
Connections:
- new net N$3: F1.2, U2.LEDA, U2.VCC
- net +3V3: now also F1.1, TP7.TP; no longer U2.VCC
- net 5V: now also TP6.TP; no longer J1.6, U2.LEDA
- net G20: now also TP2.TP; no longer J1.2
- net G21: now also TP3.TP; no longer J1.3
- net GND: now also TP1.TP; no longer J1.1
- net SCL: now also TP5.TP; no longer J1.5
- net SDA: now also TP4.TP; no longer J1.4
Other:
- moved on the sheet: Q1, R1, R2, R3, R4, R5, R6, U1, U2
